File: fork_Fan/IO_opera.kicad_sch (KiCad schematic)
At the start: 0 parts

Commit message: 完善原理图，还未完成
Parts:
- added C28: 100nF, Capacitor_SMD:C_0603_1608Metric, symbol Device:C
- added D13: APA102-2020, LED_SMD:LED-APA102-2020, symbol LED:APA102-2020
- added Q10: SS8050, Package_TO_SOT_SMD:SOT-23, symbol Transistor_BJT:SS8050
- added R30, R34, R35: 2K, Resistor_SMD:R_0603_1608Metric, symbol Device:R
- added R31: 10K, Resistor_SMD:R_0603_1608Metric, symbol Device:R
- added R32: 200K, Resistor_SMD:R_0603_1608Metric, symbol Device:R
- added R33: 100K, Resistor_SMD:R_0603_1608Metric, symbol Device:R
- added SW1, SW2: SW_Push, Button_Switch_SMD:SW_SPST_B3U-1000P, symbol Switch:SW_Push
Connections:
- new net: R30.2, SW1.1
- new net: Q10.1 (B), R31.2
- new net: R32.2, R33.1, R34.2
- new net: R35.2, SW2.1
- new net +5V: D13.1 (VDD)
- new net GND: C28.2, D13.6 (GND), Q10.2 (E), R33.2, SW1.2, SW2.2
- new net VBUS: R31.1
- new net Vbat: R32.1
- new net bat_sample: C28.1, R34.1
- new net key: R30.1
- new net sense: Q10.3 (C)
