File: fork_Fan/motor_driver.kicad_sch (KiCad schematic)
At the start: 0 parts

Commit message: add mcu and some motor driver need bat sample, key, programing pad, fuse, fd6288 power.
Parts:
- added Q2, Q3, Q4, Q5, Q6, Q7: Q_NMOS, me_Lib:PDFN-8_L3.3-W3.3-P0.65-BL-DSG, symbol Device:Q_NMOS
- added U4: FD6288Q, Package_DFN_QFN:QFN-24-1EP_4x4mm_P0.5mm_EP2.6x2.6mm, symbol my_Lib:FD6288Q_C328453
Connections:
- new net: Q6.D, Q7.S
- new net: Q4.D, Q5.S
- new net: Q2.D, Q3.S
- new net GND: Q3.D, Q5.D, Q7.D

Commit message: 完善原理图，还未完成
Parts:
- added C20, C21, C22: 10nF, Capacitor_SMD:C_0603_1608Metric, symbol Device:C
- added C23, C24, C25: 1uF, Capacitor_SMD:C_0603_1608Metric, symbol Device:C
- added C26, C27: 10uF, Capacitor_SMD:C_0603_1608Metric, symbol Device:C
- added D10, D11, D12, D14, D5, D6, D7, D8, D9: 1N5819WS, me_Lib:D_SOD-323, symbol Diode:1N5819WS
- added F1: Fuse, Fuse:Fuseholder_Littelfuse_Nano2_157x, symbol Device:Fuse
- added Q8: AO3401A, Package_TO_SOT_SMD:SOT-23, symbol Transistor_FET:AO3401A
- added Q9: SS8050, Package_TO_SOT_SMD:SOT-23, symbol Transistor_BJT:SS8050
- added R10, R11, R12, R7, R8, R9: 5.1R, Resistor_SMD:R_0603_1608Metric, symbol Device:R
- added R13, R14, R15, R16, R17, R18, R19, R20, R21, R22, R23, R24, R28: 10K, Resistor_SMD:R_0603_1608Metric, symbol Device:R
- added R25, R26, R27, R29: 2K, Resistor_SMD:R_0603_1608Metric, symbol Device:R
- added TP1, TP2, TP3: TestPoint, TestPoint:TestPoint_THTPad_D3.0mm_Drill1.5mm, symbol Connector:TestPoint
Connections:
- net GND: now also U4.6 (COM), C20.1, C21.1, C22.1, C26.2, C27.2, Q9.2 (E), R15.2, R16.2, R17.2, R25.2, R26.2, R27.2
- net A_L1: now reaches U4.1 (LIN1)
- net M_B_L2: now reaches U4.10 (LO2)
- net M_B_L2: now also D8.1 (K), R10.1
- net M_A_L1: now reaches U4.11 (LO1)
- net M_A_L1: now also D6.1 (K), R8.1
- net C: now reaches U4.12 (VS3)
- net C: now also Q6.D, Q7.S, C25.2, R18.2, R21.1, TP3.1
- net M_C_H3: now reaches U4.13 (HO3)
- net M_C_H3: now also D9.1 (K), R11.1
- net VB_C: now reaches U4.14 (VB3)
- net VB_C: now also C25.1, D12.1 (K)
- net B: now reaches U4.15 (VS2)
- net B: now also Q4.D, Q5.S, C24.2, R14.2, R20.1, TP2.1
- net M_B_H2: now reaches U4.16 (HO2)
- net M_B_H2: now also D7.1 (K), R9.1
- net VB_B: now reaches U4.17 (VB2)
- net VB_B: now also C24.1, D11.1 (K)
- net A: now reaches U4.18 (VS1)
- net A: now also Q2.D, Q3.S, C23.2, R13.2, R19.1, TP1.1
- net M_A_H1: now reaches U4.19 (HO1)
- net M_A_H1: now also D5.1 (K), R7.1
- net B_L2: now reaches U4.2 (LIN2)
- net VB_A: now reaches U4.20 (VB1)
- net VB_A: now also C23.1, D14.1 (K)
- net A_H1: now reaches U4.22 (HIN1)
- net B_H2: now reaches U4.23 (HIN2)
- net C_H3: now reaches U4.24 (HIN3)
- net C_L3: now reaches U4.3 (LIN3)
- net VDRV: now reaches U4.4 (VCC)
- net VDRV: now also C26.1, C27.1, D11.2 (A), D12.2 (A), D14.2 (A), Q8.3 (D)
- net M_C_L3: now reaches U4.9 (LO3)
- net M_C_L3: now also D10.1 (K), R12.1
- net at Q6.G: now also D9.2 (A), R11.2, R18.1
- net at Q6.S: now also Q2.S, Q4.S, F1.2
- net at Q5.G: now also D8.2 (A), R10.2, R16.1
- net at Q4.G: now also D7.2 (A), R14.1, R9.2
- net at Q3.G: now also D6.2 (A), R15.1, R8.2
- net at Q7.G: now also D10.2 (A), R12.2, R17.1
- net at Q2.G: now also D5.2 (A), R13.1, R7.2
- new net: Q9.1 (B), R29.1
- new net: Q8.1 (G), Q9.3 (C), R28.2
- new net ADC11: C20.2, R19.2, R22.1, R25.1
- new net ADC12: C21.2, R20.2, R23.1, R26.1
- new net ADC13: C22.2, R21.2, R24.1, R27.1
- new net COMP-: R22.2, R23.2, R24.2
- new net Vbat: F1.1, Q8.2 (S), R28.1
- new net switch: R29.2
Other:
- moved on the sheet: Q2, Q3, Q4, Q5, Q6, Q7, U4
