File: fork_Fan/stc_mcu.kicad_sch (KiCad schematic)
At the start: 0 parts

Commit message: add mcu and some motor driver need bat sample, key, programing pad, fuse, fd6288 power.
Parts:
- added C17, C18: 22uF, Capacitor_SMD:C_0603_1608Metric, symbol Device:C
- added C19: 100nF, Capacitor_SMD:C_0603_1608Metric, symbol Device:C
- added U3: STC8G1K08-38I-TSSOP20, Package_SO:TSSOP-20_4.4x6.5mm_P0.65mm, symbol MCU_STC:STC8G1K08-38I-TSSOP20
Connections:
- new net +5V: C17.1, C18.1, C19.1, U3.8 (VCC)
- new net GND: C17.2, C18.2, C19.2, U3.10 (GND)

Commit message: 完善原理图，还未完成
Parts:
- removed U3: STC8G1K08-38I-TSSOP20, Package_SO:TSSOP-20_4.4x6.5mm_P0.65mm, symbol MCU_STC:STC8G1K08-38I-TSSOP20
- added J3: Conn_01x04, Connector_PinHeader_2.54mm:PinHeader_1x04_P2.54mm_Vertical, symbol Connector_Generic:Conn_01x04
- added U3: STC8H1K08-38I-TSSOP20, Package_SO:TSSOP-20_4.4x6.5mm_P0.65mm, symbol my_Lib:STC8H1K08-38I-TSSOP20
Connections:
- net +5V: now also J3.1 (Pin_1), U3.8 (VCC), U3.9 (ADC_VRef+)
- net GND: now also J3.2 (Pin_2), U3.10 (GND)
- new net RX: J3.4 (Pin_4), U3.12 (TxD/ADC9/P3.1)
- new net TX: J3.3 (Pin_3), U3.11 (INT4/RxD/ADC8/P3.0)
