File: fork_Fan/fork_Fan.kicad_pcb (KiCad board)
At the start: 2 copper layers, 30 parts, among them J1 Conn_01x02, J2 USB_C_Receptacle_PowerOnly_6P, Q1 Q_NMOS, U1 CS5086E, U2 HT7150-1

Commit message: add mcu and some motor driver need bat sample, key, programing pad, fuse, fd6288 power.
Parts:
- added C16: 100nF, Capacitor_SMD:C_0603_1608Metric, F.Cu at (148.7, 121.3)
- added C17: 22uF, Capacitor_SMD:C_0603_1608Metric, F.Cu at (138.3, 116.8)
- added C18: 22uF, Capacitor_SMD:C_0603_1608Metric, F.Cu at (138.3, 119.3)
- added C19: 100nF, Capacitor_SMD:C_0603_1608Metric, F.Cu at (138.3, 121.8)
- added D4: SS54, Diode_SMD:D_SMA, F.Cu at (146.4, 117.8)
- added JP1: SolderJumper_2_Open, Jumper:SolderJumper-2_P1.3mm_Open_RoundedPad1.0x1.5mm, F.Cu at (144.5, 121.9)
- added Q2: Q_NMOS, me_Lib:PDFN-8_L3.3-W3.3-P0.65-BL-DSG, F.Cu at (129.7, 104.3)
- added Q3: Q_NMOS, me_Lib:PDFN-8_L3.3-W3.3-P0.65-BL-DSG, F.Cu at (134.6, 104.3)
- added Q4: Q_NMOS, me_Lib:PDFN-8_L3.3-W3.3-P0.65-BL-DSG, F.Cu at (139.4, 104.3)
- added Q5: Q_NMOS, me_Lib:PDFN-8_L3.3-W3.3-P0.65-BL-DSG, F.Cu at (144.3, 104.3)
- added Q6: Q_NMOS, me_Lib:PDFN-8_L3.3-W3.3-P0.65-BL-DSG, F.Cu at (149.2, 104.3)
- added Q7: Q_NMOS, me_Lib:PDFN-8_L3.3-W3.3-P0.65-BL-DSG, F.Cu at (154.1, 104.3)
- added U3: STC8G1K08-38I-TSSOP20, Package_SO:TSSOP-20_4.4x6.5mm_P0.65mm, F.Cu at (131.9, 119.6)
- added U4: FD6288Q, Package_DFN_QFN:QFN-24-1EP_4x4mm_P0.5mm_EP2.6x2.6mm, F.Cu at (130.7, 110.4)
- Q1: footprint me_Lib:PQFN-8_L6.0-W5.0-P1.27-LS6.0-BL_DSG -> me_Lib:PDFN-8_L3.3-W3.3-P0.65-BL-DSG
Connections:
- net /power_chrg/CHRG_STAT renamed /power_chrg/stat
- C12 pad 1: Vbat -> Net-(D4-K)
- C13 pad 1: Vbat -> Net-(D4-K)
- Q1 pad G: Net-(D3-K) -> Net-(JP1-A)
- R6 pad 2: Net-(D3-K) -> Net-(JP1-A)
- U2 pad 2: Vbat -> Net-(D4-K)

Commit message: fix code
Parts:
- added C20: 10nF, Capacitor_SMD:C_0603_1608Metric, F.Cu at (183.1, 103.1)
- added C21: 10nF, Capacitor_SMD:C_0603_1608Metric, F.Cu at (183.1, 105.6)
- added C22: 10nF, Capacitor_SMD:C_0603_1608Metric, F.Cu at (183.1, 108.2)
- added C23: 1uF, Capacitor_SMD:C_0603_1608Metric, F.Cu at (183.1, 110.7)
- added C24: 1uF, Capacitor_SMD:C_0603_1608Metric, F.Cu at (183.1, 113.2)
- added C25: 1uF, Capacitor_SMD:C_0603_1608Metric, F.Cu at (183.1, 115.7)
- added C26: 10uF, Capacitor_SMD:C_0603_1608Metric, F.Cu at (183.1, 118.2)
- added C27: 10uF, Capacitor_SMD:C_0603_1608Metric, F.Cu at (183.1, 120.7)
- added C28: 100nF, Capacitor_SMD:C_0603_1608Metric, F.Cu at (214.0, 103.1)
- added D10: 1N5819WS, me_Lib:D_SOD-323, F.Cu at (203.6, 124.4)
- added D11: 1N5819WS, me_Lib:D_SOD-323, F.Cu at (207.9, 118.5)
- added D12: 1N5819WS, me_Lib:D_SOD-323, F.Cu at (207.9, 121.5)
- added D13: APA102-2020, LED_SMD:LED-APA102-2020, F.Cu at (218.1, 117.1)
- added D14: 1N5819WS, me_Lib:D_SOD-323, F.Cu at (207.9, 124.4)
- added D5: 1N5819WS, me_Lib:D_SOD-323, F.Cu at (199.3, 118.5)
- added D6: 1N5819WS, me_Lib:D_SOD-323, F.Cu at (199.3, 121.5)
- added D7: 1N5819WS, me_Lib:D_SOD-323, F.Cu at (199.3, 124.4)
- added D8: 1N5819WS, me_Lib:D_SOD-323, F.Cu at (203.6, 118.5)
- added D9: 1N5819WS, me_Lib:D_SOD-323, F.Cu at (203.6, 121.5)
- added F1: Fuse, Fuse:Fuseholder_Littelfuse_Nano2_157x, F.Cu at (185.5, 124.6)
- added J3: Conn_01x04, Connector_PinHeader_2.54mm:PinHeader_1x04_P2.54mm_Vertical, F.Cu at (183.4, 131.5)
- added Q10: SS8050, Package_TO_SOT_SMD:SOT-23, F.Cu at (218.5, 112.8)
- added Q8: AO3401A, Package_TO_SOT_SMD:SOT-23, F.Cu at (204.6, 104.1)
- added Q9: SS8050, Package_TO_SOT_SMD:SOT-23, F.Cu at (204.6, 108.5)
- added R10: 5.1R, Resistor_SMD:R_0603_1608Metric, F.Cu at (187.1, 110.7)
- added R11: 5.1R, Resistor_SMD:R_0603_1608Metric, F.Cu at (187.1, 113.2)
- added R12: 5.1R, Resistor_SMD:R_0603_1608Metric, F.Cu at (187.1, 115.7)
- added R13: 10K, Resistor_SMD:R_0603_1608Metric, F.Cu at (187.1, 118.2)
- added R14: 10K, Resistor_SMD:R_0603_1608Metric, F.Cu at (187.1, 120.7)
- added R15: 10K, Resistor_SMD:R_0603_1608Metric, F.Cu at (191.1, 103.1)
- added R16: 10K, Resistor_SMD:R_0603_1608Metric, F.Cu at (191.1, 105.6)
- added R17: 10K, Resistor_SMD:R_0603_1608Metric, F.Cu at (191.1, 108.2)
- added R18: 10K, Resistor_SMD:R_0603_1608Metric, F.Cu at (191.1, 110.7)
- added R19: 10K, Resistor_SMD:R_0603_1608Metric, F.Cu at (191.1, 113.2)
- added R20: 10K, Resistor_SMD:R_0603_1608Metric, F.Cu at (191.1, 115.7)
- added R21: 10K, Resistor_SMD:R_0603_1608Metric, F.Cu at (191.1, 118.2)
- added R22: 10K, Resistor_SMD:R_0603_1608Metric, F.Cu at (191.1, 120.7)
- added R23: 10K, Resistor_SMD:R_0603_1608Metric, F.Cu at (195.1, 103.1)
- added R24: 10K, Resistor_SMD:R_0603_1608Metric, F.Cu at (195.1, 105.6)
- added R25: 2K, Resistor_SMD:R_0603_1608Metric, F.Cu at (195.1, 108.2)
- added R26: 2K, Resistor_SMD:R_0603_1608Metric, F.Cu at (195.1, 110.7)
- added R27: 2K, Resistor_SMD:R_0603_1608Metric, F.Cu at (195.1, 113.2)
- added R28: 10K, Resistor_SMD:R_0603_1608Metric, F.Cu at (195.1, 115.7)
- added R29: 2K, Resistor_SMD:R_0603_1608Metric, F.Cu at (195.1, 118.2)
- added R30: 2K, Resistor_SMD:R_0603_1608Metric, F.Cu at (214.0, 105.6)
- added R31: 10K, Resistor_SMD:R_0603_1608Metric, F.Cu at (214.0, 108.2)
- added R32: 200K, Resistor_SMD:R_0603_1608Metric, F.Cu at (214.0, 110.7)
- added R33: 100K, Resistor_SMD:R_0603_1608Metric, F.Cu at (214.0, 113.2)
- added R34: 2K, Resistor_SMD:R_0603_1608Metric, F.Cu at (214.0, 115.7)
- added R35: 2K, Resistor_SMD:R_0603_1608Metric, F.Cu at (214.0, 118.2)
- added R7: 5.1R, Resistor_SMD:R_0603_1608Metric, F.Cu at (187.1, 103.1)
- added R8: 5.1R, Resistor_SMD:R_0603_1608Metric, F.Cu at (187.1, 105.6)
- added R9: 5.1R, Resistor_SMD:R_0603_1608Metric, F.Cu at (187.1, 108.2)
- added SW1: SW_Push, Button_Switch_SMD:SW_SPST_B3U-1000P, F.Cu at (219.0, 104.0)
- added SW2: SW_Push, Button_Switch_SMD:SW_SPST_B3U-1000P, F.Cu at (219.0, 108.4)
- added TP1: TestPoint, TestPoint:TestPoint_THTPad_D3.0mm_Drill1.5mm, F.Cu at (199.7, 104.4)
- added TP2: TestPoint, TestPoint:TestPoint_THTPad_D3.0mm_Drill1.5mm, F.Cu at (199.7, 109.5)
- added TP3: TestPoint, TestPoint:TestPoint_THTPad_D3.0mm_Drill1.5mm, F.Cu at (199.7, 114.5)
- added U3: STC8H1K08-38I-TSSOP20, Package_SO:TSSOP-20_4.4x6.5mm_P0.65mm, F.Cu at (190.4, 133.2)
Connections:
- Q2 pad D: unconnected-(Q2-PadD) -> /motor_driver/A
- Q2 pad G: unconnected-(Q2-PadG) -> Net-(D5-A)
- Q2 pad S: unconnected-(Q2-PadS) -> Net-(F1-Pad2)
- Q3 pad D: unconnected-(Q3-PadD) -> GND
- Q3 pad G: unconnected-(Q3-PadG) -> Net-(D6-A)
- Q3 pad S: unconnected-(Q3-PadS) -> /motor_driver/A
- Q4 pad D: unconnected-(Q4-PadD) -> /motor_driver/B
- Q4 pad G: unconnected-(Q4-PadG) -> Net-(D7-A)
- Q4 pad S: unconnected-(Q4-PadS) -> Net-(F1-Pad2)
- Q5 pad D: unconnected-(Q5-PadD) -> GND
- Q5 pad G: unconnected-(Q5-PadG) -> Net-(D8-A)
- Q5 pad S: unconnected-(Q5-PadS) -> /motor_driver/B
- Q6 pad D: unconnected-(Q6-PadD) -> /motor_driver/C
- Q6 pad G: unconnected-(Q6-PadG) -> Net-(D9-A)
- Q6 pad S: unconnected-(Q6-PadS) -> Net-(F1-Pad2)
- Q7 pad D: unconnected-(Q7-PadD) -> GND
- Q7 pad G: unconnected-(Q7-PadG) -> Net-(D10-A)
- Q7 pad S: unconnected-(Q7-PadS) -> /motor_driver/C
- U4 pad 1: unconnected-(U4-LIN1-Pad1) -> /motor_driver/A_L1
- U4 pad 10: unconnected-(U4-LO2-Pad10) -> /motor_driver/M_B_L2
- U4 pad 11: unconnected-(U4-LO1-Pad11) -> /motor_driver/M_A_L1
- U4 pad 12: unconnected-(U4-VS3-Pad12) -> /motor_driver/C
- U4 pad 13: unconnected-(U4-HO3-Pad13) -> /motor_driver/M_C_H3
- U4 pad 14: unconnected-(U4-VB3-Pad14) -> /motor_driver/VB_C
- U4 pad 15: unconnected-(U4-VS2-Pad15) -> /motor_driver/B
- U4 pad 16: unconnected-(U4-HO2-Pad16) -> /motor_driver/M_B_H2
- U4 pad 17: unconnected-(U4-VB2-Pad17) -> /motor_driver/VB_B
- U4 pad 18: unconnected-(U4-VS1-Pad18) -> /motor_driver/A
- U4 pad 19: unconnected-(U4-HO1-Pad19) -> /motor_driver/M_A_H1
- U4 pad 2: unconnected-(U4-LIN2-Pad2) -> /motor_driver/B_L2
- U4 pad 20: unconnected-(U4-VB1-Pad20) -> /motor_driver/VB_A
- U4 pad 22: unconnected-(U4-HIN1-Pad22) -> /motor_driver/A_H1
- U4 pad 23: unconnected-(U4-HIN2-Pad23) -> /motor_driver/B_H2
- U4 pad 24: unconnected-(U4-HIN3-Pad24) -> /motor_driver/C_H3
- U4 pad 3: unconnected-(U4-LIN3-Pad3) -> /motor_driver/C_L3
- U4 pad 4: unconnected-(U4-VCC-Pad4) -> VDRV
- U4 pad 6: unconnected-(U4-COM-Pad6) -> GND
- U4 pad 9: unconnected-(U4-LO3-Pad9) -> /motor_driver/M_C_L3
